Commit message: stable slam

File: simulation/ros2_boldbot/boldbot_description/urdf/boldbot.urdf (robot description, URDF)
Before this commit: robot boldbot, 43 links, 42 joints
Links:
- removed link gaze
- added link base_footprint
- added link camera_rgb
Joints:
- added joint base_footprint_j: type fixed, parent base_footprint, child base_link, origin xyz=0.07 0 0 rpy=0 0 0
- joint head-gaze: child gaze -> camera_rgb; origin xyz=0 0 0 rpy=0 0 0 -> xyz=0 0 0 rpy=-1.57 0 -1.57

File: simulation/ros2_boldbot/boldbot_description/urdf/boldbot.urdf.xacro (robot description, xacro)
@@ -147,9 +147,9 @@
   </gazebo>
   <joint name="head-gaze" type="fixed">
-    <parent link="head" />
-    <child link="gaze" />
-    <origin xyz="0 0 0" rpy="0 0 0" />
-  </joint>
-  <link name="gaze">
+    <parent link="head"/>
+    <child link="camera_rgb"/>
+    <origin rpy="-1.57 0 -1.57" xyz="0 0 0"/>
+  </joint>
+  <link name="camera_rgb">
   </link>
   <!-- Arms -->
@@ -429,40 +429,59 @@
   <xacro:leg side="l"/>
   <xacro:leg side="r"/>
+  <joint name="base_footprint_j" type="fixed">
+    <parent link="base_footprint"/>
+    <child link="base_link"/>
+    <origin rpy="0 0 0" xyz="0.07 0 0"/>
+  </joint>
+  <link name="base_footprint">
+  </link>
   <gazebo>
-    <plugin name="boldbot_gazebo" filename="libboldbot_gazebo_plugin.so">
+    <plugin filename="libboldbot_gazebo_plugin.so" name="boldbot_gazebo">
     </plugin>
   </gazebo>
   <gazebo reference="head">
-    <sensor name='camera' type='depth'>
-      <pose>0 0 0 0 0 0</pose>
-      <camera name='__default__'>
-        <horizontal_fov>1.012300</horizontal_fov>
-        <image>
-          <width>640</width>
-          <height>480</height>
-        </image>
-        <clip>
-          <near>0.001000</near>
-          <far>100.000000</far>
-        </clip>
-      </camera>
-      <always_on>1</always_on>
-      <update_rate>30</update_rate>
-      <visualize>true</visualize>
-      <plugin name="camera_controller" filename="libgazebo_ros_camera.so">
-        <alwaysOn>true</alwaysOn>
-        <updateRate>30</updateRate>
-        <imageTopicName>image</imageTopicName>
-        <cameraInfoTopicName>camera_info</cameraInfoTopicName>
-        <depthImageTopicName>depth/image</depthImageTopicName>
-        <frameName>camera_link</frameName>
-        <hackBaseline>0.07</hackBaseline>
-        <distortionK1>0.0</distortionK1>
-        <distortionK2>0.0</distortionK2>
-        <distortionK3>0.0</distortionK3>
-        <distortionT1>0.0</distortionT1>
-        <distortionT2>0.0</distortionT2>
-      </plugin>
-    </sensor>
+      <sensor name="camera_depth" type="depth">
+        <always_on>1</always_on>
+        <update_rate>1</update_rate>
+        <pose>0 0 0 0 0 0</pose>
+        <camera name="camera_depth">
+        </camera>
+	          <plugin name="camera_driver" filename="libgazebo_ros_camera.so">
+            <camera_name>camera_depth</camera_name>
+            <frame_name>camera_depth</frame_name>
+            <hack_baseline>0.07</hack_baseline>
+            <min_depth>0.001</min_depth>
+          </plugin>
+      </sensor>
+  </gazebo>
+  <gazebo reference="head">
+      <sensor name="camera_rgb" type="camera">
+        <always_on>true</always_on>
+        <visualize>true</visualize>
+        <update_rate>30</update_rate>
+	      <pose>0 0 0 0 0 0</pose>
+        <camera name="camera_rgb">
+          <horizontal_fov>1.02974</horizontal_fov>
+          <image>
+            <width>320</width>
+            <height>240</height>
+            <format>R8G8B8</format>
+          </image>
+          <clip>
+            <near>0.02</near>
+            <far>300</far>
+          </clip>
+          <noise>
+            <type>gaussian</type>
+            <mean>0.0</mean>
+            <stddev>0.007</stddev>
+          </noise>
+        </camera>
+          <plugin name="camera_driver" filename="libgazebo_ros_camera.so">
+            <camera_name>camera_rgb</camera_name>
+            <frame_name>camera_rgb</frame_name>
+            <hack_baseline>0.07</hack_baseline>
+          </plugin>
+      </sensor>
   </gazebo>
  <gazebo reference="torso">
@@ -483,12 +502,18 @@
     </sensor>
   </gazebo>
-  <!-- <gazebo>
-    <plugin name="object_controller" filename="libgazebo_ros_planar_move.so">
-      <commandTopic>cmd_vel</commandTopic>
-      <odometryTopic>odom</odometryTopic>
-      <odometryFrame>odom</odometryFrame>
-      <odometryRate>20.0</odometryRate>
-      <robotBaseFrame>base_link</robotBaseFrame>
+  <gazebo>
+    <plugin filename="libgazebo_ros_planar_move.so" name="object_controller">
+      <ros>
+        <!-- <argument>cmd_vel:=custom_cmd_vel</argument> -->
+        <argument>odom:=odom_cmd</argument>
+      </ros>
+      <publish_odom>true</publish_odom>
+      <publish_odom_tf>false</publish_odom_tf>
+      <odometry_frame>odom_demo</odometry_frame>
+      <robot_base_frame>base_link</robot_base_frame>
+      <covariance_x>0.0001</covariance_x>
+      <covariance_y>0.0001</covariance_y>
+      <covariance_yaw>0.01</covariance_yaw>
     </plugin>
-  </gazebo> -->
+  </gazebo>
 </robot>

Commit message: stable humble

File: simulation/ros2_boldbot/boldbot_description/urdf/boldbot.urdf (robot description, URDF)
Before this commit: robot boldbot, 44 links, 43 joints
Links:
- removed link camera_rgb
- added link camera_depth
Joints:
- joint head-gaze: child camera_rgb -> camera_depth

File: simulation/ros2_boldbot/boldbot_description/urdf/boldbot.urdf.xacro (robot description, xacro)
@@ -148,8 +148,8 @@
   <joint name="head-gaze" type="fixed">
     <parent link="head"/>
-    <child link="camera_rgb"/>
+    <child link="camera_depth"/>
     <origin rpy="-1.57 0 -1.57" xyz="0 0 0"/>
   </joint>
-  <link name="camera_rgb">
+  <link name="camera_depth">
   </link>
   <!-- Arms -->
@@ -511,5 +511,5 @@
       <publish_odom_tf>false</publish_odom_tf>
       <odometry_frame>odom_demo</odometry_frame>
-      <robot_base_frame>base_link</robot_base_frame>
+      <robot_base_frame>base_footprint</robot_base_frame>
       <covariance_x>0.0001</covariance_x>
       <covariance_y>0.0001</covariance_y>

File: simulation/ros2_boldbot/boldbot_description/urdf/boldbot_nav.urdf (robot description, URDF)
Before this commit: robot boldbot, 44 links, 43 joints
Links:
- removed link camera_rgb
- added link camera_depth
Joints:
- joint head-gaze: child camera_rgb -> camera_depth

File: simulation/simulation/description/depth_camera.xacro (robot description, xacro)
@@ -16,8 +16,8 @@
     <joint name="camera_optical_joint" type="fixed">
         <parent link="camera_link"/>
-        <child link="camera_rgb"/>
+        <child link="camera_depth"/>
         <origin xyz="0 0 0" rpy="${-pi/2} 0 ${-pi/2}"/>
     </joint>
-    <link name="camera_rgb"></link>
+    <link name="camera_depth"></link>
     <gazebo reference="camera_link">
         <sensor name="camera_depth" type="depth">

File: simulation/simulation/description/gazebo_control.xacro (robot description, xacro)
@@ -13,8 +13,8 @@
             <!-- Output -->
             <odometry_frame>odom</odometry_frame>
-            <robot_base_frame>base_link</robot_base_frame>
+            <robot_base_frame>base_footprint</robot_base_frame>
             <publish_odom>true</publish_odom>
-            <publish_odom_tf>true</publish_odom_tf>
-            <publish_wheel_tf>true</publish_wheel_tf>
+            <publish_odom_tf>false</publish_odom_tf>
+            <publish_wheel_tf>false</publish_wheel_tf>
         </plugin>
     </gazebo>

File: simulation/simulation/description/robot_core.xacro (robot description, xacro)
@@ -36,6 +36,6 @@
     <!-- BASE_FOOTPRINT LINK -->
     <joint name="base_footprint_joint" type="fixed">
-        <parent link="base_link"/>
-        <child link="base_footprint"/>
+        <parent link="base_footprint"/>
+        <child link="base_link"/>
         <origin xyz="0 0 0" rpy="0 0 0"/>
     </joint>
