Commit message: update to slam

File: simulation/ros2_boldbot/boldbot_description/urdf/boldbot_nav.urdf (robot description, URDF)
Before this commit: robot boldbot, 43 links, 42 joints
Links:
- removed link gaze
- added link camera
Joints:
- joint head-gaze: child gaze -> camera

Commit message: develop rtabmap

File: simulation/ros2_boldbot/boldbot_description/urdf/boldbot_nav.urdf (robot description, URDF)
Before this commit: robot boldbot, 43 links, 42 joints
Links:
- removed link camera
- added link base_footprint
- added link camera_rgb
Joints:
- added joint base_footprint_j: type fixed, parent base_footprint, child base_link, origin xyz=0.07 0 0 rpy=0 0 0
- joint head-gaze: child camera -> camera_rgb; origin xyz=0 0 0 rpy=0 0 0 -> xyz=0 0 0 rpy=-1.57 0 -1.57

Commit message: integrate free fleet

File: simulation/ros2_boldbot/boldbot_description/urdf/boldbot_nav.urdf (robot description, URDF)
Before this commit: robot boldbot, 44 links, 43 joints
Joints:
- joint head-tilt-head: origin xyz=0.065 0 0 rpy=1.5707963267948966 0 1.5707963267948966 -> xyz=0.065 0 0 rpy=1.5707963267948966 0 1.7707963267948966
